File: milight_to_485.kicad_pcb (KiCad board)
At the start: 2 copper layers, 50 x 50 mm, 29 parts, among them J1 RJ12, J2 RJ45, P1 SWIM, P2 CONN_01X02, P3 TTL, P4 TTL_SW, SW1 reset, U1 LT8900, U2 STM8S103F3, U3 MAX487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

Commit message: small changes
Parts:
- added REF**: MountingHole_3.2mm_M3, Mounting_Holes:MountingHole_3.2mm_M3, F.Cu at (125.0, 52.2)
- RST: renamed from SW1; footprint Buttons_Switches_SMD:SW_SPST_FSMSM -> BK_Common:SW_SPST_TACT_SMD_3X6
- moved ? 4.57 mm to (121.5, 58.0)
Other:
- board text added: "485"
- board text added: "TTL"

Commit message: gerber
Routing:
- net +5V: track 91.0 -> 107.7 mm
- net /485_B: track 7.04 -> 11.3 mm
- net GND: track 71.6 -> 67.4 mm, vias 6 -> 7
- net /485_A: track 9.02 -> 6.90 mm
